File: BrightBoard1/BrightBoard1.kicad_pcb (KiCad board)
At the start: 2 copper layers, 292.1 x 209.6 mm, 156 parts, among them J1 Conn_ARM_JTAG_SWD_10, J2 VIN_JACK, Q1 DMN3404L, Q2 DMN3404L, U1 E73-2G4M04S-52832, U2 TPS62177DQC

Commit message: Renamed all LEDs
Parts:
- removed the D9 at (169.5, 287.7)
- removed D?: LED_2, LED:2835_LED
- D100, D101, D102, D103, D104, D34, D35, D36, D37, D38, D39, D40, D50, D51, D52, D53, D54, D55, D56, D66, D67, D68, D69, D70, D71, D72, D82, D83, D84, D85, D86, D87, D88, D9, D98, D99: renamed from D?; value LED_2 -> LED_1
- D105, D18, D19, D2, D20, D21, D22, D23, D24, D25, D3, D4, D41, D5, D57, D6, D7, D73, D8, D89: value LED_2 -> LED_1
- gave numbers to parts that had none: 42
Connections:
- D10 pad 1: (no net) -> Net-(D10-Pad1)
- D10 pad 2: (no net) -> VCC
- D100 pad 1: (no net) -> Net-(D100-Pad1)
- D100 pad 2: (no net) -> Net-(D100-Pad2)
- D101 pad 1: (no net) -> Net-(D101-Pad1)
- D101 pad 2: (no net) -> Net-(D100-Pad1)
- D102 pad 1: (no net) -> Net-(D102-Pad1)
- D102 pad 2: (no net) -> Net-(D101-Pad1)
- D103 pad 1: (no net) -> Net-(D103-Pad1)
- D103 pad 2: (no net) -> Net-(D102-Pad1)
- D104 pad 1: (no net) -> Net-(D104-Pad1)
- D104 pad 2: (no net) -> Net-(D103-Pad1)
- D105 pad 1: (no net) -> /LEDs/STRIP_1_RETURN
- D105 pad 2: (no net) -> Net-(D104-Pad1)
- D106 pad 1: (no net) -> Net-(D106-Pad1)
- D106 pad 2: (no net) -> VCC
- D107 pad 1: (no net) -> Net-(D107-Pad1)
- D107 pad 2: (no net) -> Net-(D106-Pad1)
- D108 pad 1: (no net) -> Net-(D108-Pad1)
- D108 pad 2: (no net) -> Net-(D107-Pad1)
- D109 pad 1: (no net) -> Net-(D109-Pad1)
- D109 pad 2: (no net) -> Net-(D108-Pad1)
- D11 pad 1: (no net) -> Net-(D11-Pad1)
- D11 pad 2: (no net) -> Net-(D10-Pad1)
- D110 pad 1: (no net) -> Net-(D110-Pad1)
- D110 pad 2: (no net) -> Net-(D109-Pad1)
- D111 pad 1: (no net) -> Net-(D111-Pad1)
- D111 pad 2: (no net) -> Net-(D110-Pad1)
- D112 pad 1: (no net) -> Net-(D112-Pad1)
- D112 pad 2: (no net) -> Net-(D111-Pad1)
- D113 pad 1: (no net) -> /LEDs/STRIP_2_RETURN
- D113 pad 2: (no net) -> Net-(D112-Pad1)
- D12 pad 1: (no net) -> Net-(D12-Pad1)
- D12 pad 2: (no net) -> Net-(D11-Pad1)
- D13 pad 1: (no net) -> Net-(D13-Pad1)
- D13 pad 2: (no net) -> Net-(D12-Pad1)
- D14 pad 1: (no net) -> Net-(D14-Pad1)
- D14 pad 2: (no net) -> Net-(D13-Pad1)
- D15 pad 1: (no net) -> Net-(D15-Pad1)
- D15 pad 2: (no net) -> Net-(D14-Pad1)
- D16 pad 1: (no net) -> Net-(D16-Pad1)
- D16 pad 2: (no net) -> Net-(D15-Pad1)
- D17 pad 1: (no net) -> /LEDs/STRIP_2_RETURN
- D17 pad 2: (no net) -> Net-(D16-Pad1)
- D18 pad 1: (no net) -> Net-(D18-Pad1)
- D18 pad 2: (no net) -> VCC
- D19 pad 1: (no net) -> Net-(D19-Pad1)
- D19 pad 2: (no net) -> Net-(D18-Pad1)
- D2 pad 1: (no net) -> Net-(D2-Pad1)
- D2 pad 2: (no net) -> VCC
- D20 pad 1: (no net) -> Net-(D20-Pad1)
- D20 pad 2: (no net) -> Net-(D19-Pad1)
- D21 pad 1: (no net) -> Net-(D21-Pad1)
- D21 pad 2: (no net) -> Net-(D20-Pad1)
- D22 pad 1: (no net) -> Net-(D22-Pad1)
- D22 pad 2: (no net) -> Net-(D21-Pad1)
- D23 pad 1: (no net) -> Net-(D23-Pad1)
- D23 pad 2: (no net) -> Net-(D22-Pad1)
- D24 pad 1: (no net) -> Net-(D24-Pad1)
- D24 pad 2: (no net) -> Net-(D23-Pad1)
- D25 pad 1: (no net) -> /LEDs/STRIP_1_RETURN
- D25 pad 2: (no net) -> Net-(D24-Pad1)
- D26 pad 1: (no net) -> Net-(D26-Pad1)
- D26 pad 2: (no net) -> VCC
- D27 pad 1: (no net) -> Net-(D27-Pad1)
- D27 pad 2: (no net) -> Net-(D26-Pad1)
- D28 pad 1: (no net) -> Net-(D28-Pad1)
- D28 pad 2: (no net) -> Net-(D27-Pad1)
- D29 pad 1: (no net) -> Net-(D29-Pad1)
- D29 pad 2: (no net) -> Net-(D28-Pad1)
- D3 pad 1: (no net) -> Net-(D3-Pad1)
- D3 pad 2: (no net) -> Net-(D2-Pad1)
- D30 pad 1: (no net) -> Net-(D30-Pad1)
- D30 pad 2: (no net) -> Net-(D29-Pad1)
- D31 pad 1: (no net) -> Net-(D31-Pad1)
- D31 pad 2: (no net) -> Net-(D30-Pad1)
- D32 pad 1: (no net) -> Net-(D32-Pad1)
- D32 pad 2: (no net) -> Net-(D31-Pad1)
- D33 pad 1: (no net) -> /LEDs/STRIP_2_RETURN
- D33 pad 2: (no net) -> Net-(D32-Pad1)
- D34 pad 1: (no net) -> Net-(D34-Pad1)
- D34 pad 2: (no net) -> VCC
- D35 pad 1: (no net) -> Net-(D35-Pad1)
- D35 pad 2: (no net) -> Net-(D34-Pad1)
- D36 pad 1: (no net) -> Net-(D36-Pad1)
- D36 pad 2: (no net) -> Net-(D35-Pad1)
- D37 pad 1: (no net) -> Net-(D37-Pad1)
- D37 pad 2: (no net) -> Net-(D36-Pad1)
- D38 pad 1: (no net) -> Net-(D38-Pad1)
- D38 pad 2: (no net) -> Net-(D37-Pad1)
- D39 pad 1: (no net) -> Net-(D39-Pad1)
- D39 pad 2: (no net) -> Net-(D38-Pad1)
- D4 pad 1: (no net) -> Net-(D4-Pad1)
- D4 pad 2: (no net) -> Net-(D3-Pad1)
- D40 pad 1: (no net) -> Net-(D40-Pad1)
- D40 pad 2: (no net) -> Net-(D39-Pad1)
- D41 pad 1: (no net) -> /LEDs/STRIP_1_RETURN
- D41 pad 2: (no net) -> Net-(D40-Pad1)
- D42 pad 1: (no net) -> Net-(D42-Pad1)
- D42 pad 2: (no net) -> VCC
- D43 pad 1: (no net) -> Net-(D43-Pad1)
- D43 pad 2: (no net) -> Net-(D42-Pad1)
- D44 pad 1: (no net) -> Net-(D44-Pad1)
- D44 pad 2: (no net) -> Net-(D43-Pad1)
- D45 pad 1: (no net) -> Net-(D45-Pad1)
- D45 pad 2: (no net) -> Net-(D44-Pad1)
- D46 pad 1: (no net) -> Net-(D46-Pad1)
- D46 pad 2: (no net) -> Net-(D45-Pad1)
- D47 pad 1: (no net) -> Net-(D47-Pad1)
- D47 pad 2: (no net) -> Net-(D46-Pad1)
- D48 pad 1: (no net) -> Net-(D48-Pad1)
- D48 pad 2: (no net) -> Net-(D47-Pad1)
- D49 pad 1: (no net) -> /LEDs/STRIP_2_RETURN
- D49 pad 2: (no net) -> Net-(D48-Pad1)
- D5 pad 1: (no net) -> Net-(D5-Pad1)
- D5 pad 2: (no net) -> Net-(D4-Pad1)
- D50 pad 1: (no net) -> Net-(D50-Pad1)
- D50 pad 2: (no net) -> VCC
- D51 pad 1: (no net) -> Net-(D51-Pad1)
- D51 pad 2: (no net) -> Net-(D50-Pad1)
- D52 pad 1: (no net) -> Net-(D52-Pad1)
- D52 pad 2: (no net) -> Net-(D51-Pad1)
- D53 pad 1: (no net) -> Net-(D53-Pad1)
- D53 pad 2: (no net) -> Net-(D52-Pad1)
- D54 pad 1: (no net) -> Net-(D54-Pad1)
- D54 pad 2: (no net) -> Net-(D53-Pad1)
- D55 pad 1: (no net) -> Net-(D55-Pad1)
- D55 pad 2: (no net) -> Net-(D54-Pad1)
- D56 pad 1: (no net) -> Net-(D56-Pad1)
- D56 pad 2: (no net) -> Net-(D55-Pad1)
- D57 pad 1: (no net) -> /LEDs/STRIP_1_RETURN
- D57 pad 2: (no net) -> Net-(D56-Pad1)
- D58 pad 1: (no net) -> Net-(D58-Pad1)
- D58 pad 2: (no net) -> VCC
- D59 pad 1: (no net) -> Net-(D59-Pad1)
- D59 pad 2: (no net) -> Net-(D58-Pad1)
- D6 pad 1: (no net) -> Net-(D6-Pad1)
- D6 pad 2: (no net) -> Net-(D5-Pad1)
- D60 pad 1: (no net) -> Net-(D60-Pad1)
- D60 pad 2: (no net) -> Net-(D59-Pad1)
- D61 pad 1: (no net) -> Net-(D61-Pad1)
- D61 pad 2: (no net) -> Net-(D60-Pad1)
- D62 pad 1: (no net) -> Net-(D62-Pad1)
- D62 pad 2: (no net) -> Net-(D61-Pad1)
- D63 pad 1: (no net) -> Net-(D63-Pad1)
- D63 pad 2: (no net) -> Net-(D62-Pad1)
- D64 pad 1: (no net) -> Net-(D64-Pad1)
- D64 pad 2: (no net) -> Net-(D63-Pad1)
- D65 pad 1: (no net) -> /LEDs/STRIP_2_RETURN
- D65 pad 2: (no net) -> Net-(D64-Pad1)
- D66 pad 1: (no net) -> Net-(D66-Pad1)
- D66 pad 2: (no net) -> VCC
- D67 pad 1: (no net) -> Net-(D67-Pad1)
- D67 pad 2: (no net) -> Net-(D66-Pad1)
- D68 pad 1: (no net) -> Net-(D68-Pad1)
- D68 pad 2: (no net) -> Net-(D67-Pad1)
- D69 pad 1: (no net) -> Net-(D69-Pad1)
- D69 pad 2: (no net) -> Net-(D68-Pad1)
- D7 pad 1: (no net) -> Net-(D7-Pad1)
- D7 pad 2: (no net) -> Net-(D6-Pad1)
- D70 pad 1: (no net) -> Net-(D70-Pad1)
- D70 pad 2: (no net) -> Net-(D69-Pad1)
- D71 pad 1: (no net) -> Net-(D71-Pad1)
- D71 pad 2: (no net) -> Net-(D70-Pad1)
- D72 pad 1: (no net) -> Net-(D72-Pad1)
- D72 pad 2: (no net) -> Net-(D71-Pad1)
- D73 pad 1: (no net) -> /LEDs/STRIP_1_RETURN
- D73 pad 2: (no net) -> Net-(D72-Pad1)
- D74 pad 1: (no net) -> Net-(D74-Pad1)
- D74 pad 2: (no net) -> VCC
- D75 pad 1: (no net) -> Net-(D75-Pad1)
- D75 pad 2: (no net) -> Net-(D74-Pad1)
- D76 pad 1: (no net) -> Net-(D76-Pad1)
- D76 pad 2: (no net) -> Net-(D75-Pad1)
- D77 pad 1: (no net) -> Net-(D77-Pad1)
- D77 pad 2: (no net) -> Net-(D76-Pad1)
- D78 pad 1: (no net) -> Net-(D78-Pad1)
- D78 pad 2: (no net) -> Net-(D77-Pad1)
- D79 pad 1: (no net) -> Net-(D79-Pad1)
- D79 pad 2: (no net) -> Net-(D78-Pad1)
- D8 pad 1: (no net) -> Net-(D8-Pad1)
- D8 pad 2: (no net) -> Net-(D7-Pad1)
- D80 pad 1: (no net) -> Net-(D80-Pad1)
- D80 pad 2: (no net) -> Net-(D79-Pad1)
- D81 pad 1: (no net) -> /LEDs/STRIP_2_RETURN
- D81 pad 2: (no net) -> Net-(D80-Pad1)
- D82 pad 1: (no net) -> Net-(D82-Pad1)
- D82 pad 2: (no net) -> VCC
- D83 pad 1: (no net) -> Net-(D83-Pad1)
- D83 pad 2: (no net) -> Net-(D82-Pad1)
- D84 pad 1: (no net) -> Net-(D84-Pad1)
- D84 pad 2: (no net) -> Net-(D83-Pad1)
- D85 pad 1: (no net) -> Net-(D85-Pad1)
- D85 pad 2: (no net) -> Net-(D84-Pad1)
- D86 pad 1: (no net) -> Net-(D86-Pad1)
- D86 pad 2: (no net) -> Net-(D85-Pad1)
- D87 pad 1: (no net) -> Net-(D87-Pad1)
- D87 pad 2: (no net) -> Net-(D86-Pad1)
- D88 pad 1: (no net) -> Net-(D88-Pad1)
- D88 pad 2: (no net) -> Net-(D87-Pad1)
- D89 pad 1: (no net) -> /LEDs/STRIP_1_RETURN
- D89 pad 2: (no net) -> Net-(D88-Pad1)
- D9 pad 1: (no net) -> /LEDs/STRIP_1_RETURN
- D9 pad 2: (no net) -> Net-(D8-Pad1)
- D90 pad 1: (no net) -> Net-(D90-Pad1)
- D90 pad 2: (no net) -> VCC
- D91 pad 1: (no net) -> Net-(D91-Pad1)
- D91 pad 2: (no net) -> Net-(D90-Pad1)
- D92 pad 1: (no net) -> Net-(D92-Pad1)
- D92 pad 2: (no net) -> Net-(D91-Pad1)
- D93 pad 1: (no net) -> Net-(D93-Pad1)
- D93 pad 2: (no net) -> Net-(D92-Pad1)
- D94 pad 1: (no net) -> Net-(D94-Pad1)
- D94 pad 2: (no net) -> Net-(D93-Pad1)
- D95 pad 1: (no net) -> Net-(D95-Pad1)
- D95 pad 2: (no net) -> Net-(D94-Pad1)
- D96 pad 1: (no net) -> Net-(D96-Pad1)
- D96 pad 2: (no net) -> Net-(D95-Pad1)
- D97 pad 1: (no net) -> /LEDs/STRIP_2_RETURN
- D97 pad 2: (no net) -> Net-(D96-Pad1)
- D98 pad 1: (no net) -> Net-(D98-Pad1)
- D98 pad 2: (no net) -> VCC
- D99 pad 1: (no net) -> Net-(D100-Pad2)
- D99 pad 2: (no net) -> Net-(D98-Pad1)

Commit message: Added mounting holes
Parts:
- moved MH4 240.5 mm to (258.4, 297.8)
- moved MH2 239.8 mm to (258.4, 221.6)
- moved MH8 170.2 mm to (338.5, 297.8)
- moved MH6 169.2 mm to (338.5, 221.6)
Changed lines of the file:
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@@
   )
   (module MountingHole:MountingHole_4.3mm_M4_ISO14580_Pad (layer F.Cu)
-    (at 496.157001 252.822001)
+    (at 258.445 221.615)
     (descr "Mounting Hole 4.3mm, M4, ISO14580")
     (tags "mounting hole 4.3mm m4 iso14580")
@@
   )
   (module MountingHole:MountingHole_4.3mm_M4_ISO14580_Pad (layer F.Cu)
-    (at 496.157001 261.372001)
+    (at 258.445 297.815)
     (descr "Mounting Hole 4.3mm, M4, ISO14580")
     (tags "mounting hole 4.3mm m4 iso14580")
@@
   )
   (module MountingHole:MountingHole_4.3mm_M4_ISO14580_Pad (layer F.Cu)
-    (at 504.707001 252.822001)
+    (at 338.455 221.615)
     (descr "Mounting Hole 4.3mm, M4, ISO14580")
     (tags "mounting hole 4.3mm m4 iso14580")
@@
   )
   (module MountingHole:MountingHole_4.3mm_M4_ISO14580_Pad (layer F.Cu)
-    (at 504.707001 261.372001)
+    (at 338.455 297.815)
     (descr "Mounting Hole 4.3mm, M4, ISO14580")
     (tags "mounting hole 4.3mm m4 iso14580")

Commit message: Layed out LEDs, 3.3v regulator; going to change it to a larger package
Parts:
- moved D113 312.0 mm to (169.5, 111.9), turned to 270 degrees
- moved D9 312.0 mm to (427.4, 111.9), turned to 270 degrees
- moved D106 311.5 mm to (169.5, 287.2), turned to 270 degrees
- moved D2 311.5 mm to (427.4, 287.2), turned to 270 degrees
- moved D112 286.8 mm to (169.5, 137.0), turned to 270 degrees
- moved D8 286.8 mm to (427.4, 137.0), turned to 270 degrees
- moved D107 286.4 mm to (169.5, 262.2), turned to 270 degrees
- moved D3 286.4 mm to (427.4, 262.2), turned to 270 degrees
- moved D105 280.1 mm to (189.4, 111.9), turned to 270 degrees
- moved D17 280.1 mm to (407.5, 111.9), turned to 270 degrees
- moved D10 279.5 mm to (407.5, 287.2), turned to 270 degrees
- moved D98 279.5 mm to (189.4, 287.2), turned to 270 degrees
- moved D111 268.7 mm to (169.5, 162.0), turned to 270 degrees
- moved D7 268.7 mm to (427.4, 162.0), turned to 270 degrees
- moved D108 268.4 mm to (169.5, 237.1), turned to 270 degrees
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Routing:
- net /LEDs/STRIP_2_RETURN: track 0.00 -> 286.4 mm
- net VCC: track 0.00 -> 277.0 mm
- net Net-(D95-Pad1): track 0.00 -> 14.6 mm
- net Net-(D94-Pad1): track 0.00 -> 14.6 mm
- net Net-(D91-Pad1): track 0.00 -> 14.6 mm
- net Net-(D87-Pad1): track 0.00 -> 14.6 mm
- net Net-(D86-Pad1): track 0.00 -> 14.6 mm
- net Net-(D83-Pad1): track 0.00 -> 14.6 mm
- net Net-(D79-Pad1): track 0.00 -> 14.6 mm
- net Net-(D78-Pad1): track 0.00 -> 14.6 mm
- net Net-(D75-Pad1): track 0.00 -> 14.6 mm
- net Net-(D71-Pad1): track 0.00 -> 14.6 mm
- net Net-(D70-Pad1): track 0.00 -> 14.6 mm
- net Net-(D7-Pad1): track 0.00 -> 14.6 mm
- net Net-(D67-Pad1): track 0.00 -> 14.6 mm
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- added copper zone on B.Cu, net Net-(C10-Pad1)
- added copper zone on B.Cu, net Net-(C7-Pad1)
- added copper zone on B.Cu, net Net-(L1-Pad1)
Other:
- net class Default: trace_width 0.25 -> 2.54
- net class High Current added: clearance 0.2, trace_width 3.81, via_dia 0.8, via_drill 0.4
- net class Signal added: clearance 0.2, trace_width 1.016, via_dia 0.8, via_drill 0.4

Commit message: Moving over?
Parts:
- JP2, JP3: moved to F.Cu
- moved JP3 273.5 mm to (159.8, 109.9)
- moved JP2 246.7 mm to (180.1, 109.9)
- moved Q1 239.4 mm to (195.8, 123.8), turned to 90 degrees
- moved R4 238.4 mm to (194.8, 132.5), turned to 90 degrees
- moved R5 237.6 mm to (177.3, 128.1), turned to 180 degrees
- moved R2 236.5 mm to (197.6, 132.5), turned to 270 degrees
- moved C4 236.2 mm to (177.3, 137.2), turned to 180 degrees
- moved C3 236.1 mm to (193.8, 137.2), turned to 180 degrees
- moved Q2 228.5 mm to (179.7, 123.8), turned to 90 degrees
- moved R3 227.0 mm to (193.8, 128.1), turned to 180 degrees
- moved R6 215.1 mm to (178.3, 132.6), turned to 90 degrees
- moved R7 212.2 mm to (181.5, 132.6), turned to 270 degrees
- moved D1 96.2 mm to (208.7, 291.1), turned to 180 degrees
- moved C1 95.3 mm to (208.1, 269.8), turned to 90 degrees
- moved R1 93.8 mm to (204.1, 291.1)
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Connections:
- R10 pad 1: VCC -> Net-(C7-Pad1)
Routing:
- net /STRIP_2_AI: track 0.00 -> 183.3 mm, vias 0 -> 2
- net /STRIP_1_AI: track 0.00 -> 170.4 mm, vias 0 -> 2
- net /STRIP_2_EN: track 0.00 -> 161.1 mm, vias 0 -> 2
- net /STRIP_1_EN: track 0.00 -> 149.9 mm, vias 0 -> 2
- net +3V3: track 0.00 -> 56.7 mm
- net /VCC_AI: track 0.00 -> 43.4 mm, vias 0 -> 2
- net /~RESET: track 0.00 -> 34.1 mm
- net /TRACEDATA[0]: track 0.00 -> 32.1 mm, vias 0 -> 2
- net Net-(C10-Pad1): track 4.62 -> 17.4 mm, vias 0 -> 2
- net /LEDs/STRIP_1_RETURN: track 0.00 -> 9.85 mm
- net /LEDs/STRIP_2_RETURN: track 286.4 -> 295.9 mm
- net /SWDCLK: track 0.00 -> 9.06 mm
- net Net-(C7-Pad1): track 0.00 -> 8.70 mm
- net /HEARTBEAT: track 0.00 -> 7.28 mm
- net Net-(Q2-Pad1): track 0.00 -> 7.08 mm
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- added copper zone on B.Cu, net GND
Other:
- net class Signal: trace_width 1.016 -> 0.508

Commit message: Routed all traces; need to finish ESD ring
Parts:
- added MH1 (x2): M4, MountingHole:MountingHole_4.3mm_M4_ISO14580_Pad, F.Cu at (5.08, -5.08)
- moved JP2 4.06 mm to (180.1, 105.8)
Routing:
- net /LEDs/STRIP_1_RETURN: track 9.85 -> 9.12 mm, vias 0 -> 56
- net GND: vias 118 -> 224
- net /LEDs/STRIP_2_RETURN: vias 0 -> 8
- net (no net): vias 0 -> 16
- added copper zone on B.Cu, net /LEDs/STRIP_1_RETURN
- added copper zone on B.Cu, net /LEDs/STRIP_2_RETURN

Commit message: Finished
Parts:
- removed the MH1 at (5.08, -5.08) (x2)
- added G***: LOGO, BrightBoard:logo, B.Cu at (297.3, 171.7)
- moved J2 3.04 mm to (241.0, 293.7)
Connections:
- J1 pad 7: Net-(J1-Pad7) -> (no net)
- J1 pad 8: Net-(J1-Pad8) -> (no net)
- U1 pad 10: /P0.30 -> (no net)
- U1 pad 11: /P0.31 -> (no net)
- U1 pad 12: Net-(U1-Pad12) -> (no net)
- U1 pad 13: Net-(U1-Pad13) -> (no net)
- U1 pad 14: Net-(U1-Pad14) -> (no net)
- U1 pad 20: /P0.05 -> (no net)
- U1 pad 23: /P0.08 -> (no net)
- U1 pad 24: /P0.09 -> (no net)
- U1 pad 25: /P0.10 -> (no net)
- U1 pad 26: /P0.11 -> (no net)
- U1 pad 27: /P0.12 -> (no net)
- U1 pad 28: /P0.13 -> (no net)
- U1 pad 29: /TRACEDATA[3] -> (no net)
- U1 pad 3: Net-(U1-Pad3) -> (no net)
- U1 pad 30: /TRACEDATA[2] -> (no net)
- U1 pad 31: /TRACEDATA[1] -> (no net)
- U1 pad 34: /P0.19 -> (no net)
- U1 pad 35: /TRACECLK -> (no net)
- U1 pad 39: /P0.22 -> (no net)
- U1 pad 4: Net-(U1-Pad4) -> (no net)
- U1 pad 40: /P0.23 -> (no net)
- U1 pad 41: /P0.24 -> (no net)
- U1 pad 5: /P0.25 -> (no net)
- U1 pad 6: /P0.26 -> (no net)
- U1 pad 7: /P0.27 -> (no net)
- U1 pad 8: /P0.28 -> (no net)
- U1 pad 9: /P0.29 -> (no net)
Routing:
- net VCC: track 274.7 -> 291.7 mm
- net GND: vias 224 -> 297
- net (no net): vias 16 -> 0
Other:
- board text added: "Bluetooth Communication + 3.3V Power"
- board text added: "Input: 24V +/- 5% Power: 50W Nominal, 67.2W Max Efficiency: 167 - 142 Lumens/W 7100 - 11200 Lumens"
- board text added: "Power Transistors + Current Sense"
- board text added: "Version 1.0 By Vlad Pomogaev"
